File: $DCMGv2_SIGNALROUTING.sch (KiCad schematic (older format))
At the start: 320 parts, among them P1 BRANCH 1 BUS 1 LOAD3 NC, P10 BRANCH 1 BUS 1 LOAD 2 NC, P100 CONNECTOR, P101 CONNECTOR, P102 CONNECTOR, P103 CONNECTOR, P104 CONNECTOR, P105 CONNECTOR, P106 CONNECTOR, P107 CONNECTOR, P108 CONNECTOR, P109 CONNECTOR, P11 BRANCH 1 BUS 1 LOAD 1 NO, P110 CONNECTOR, P111 CONNECTOR, P112 CONNECTOR, P113 CONNECTOR, P114 CONNECTOR, P115 CONNECTOR, P116 CONNECTOR, P117 CONNECTOR, P118 CONNECTOR, P119 CONNECTOR, P12 BRANCH 1 BUS 1 LOAD 1 NC, P120 CONNECTOR, P121 CONNECTOR, P122 CONNECTOR, P123 CONNECTOR, P124 CONNECTOR, P125 CONNECTOR, P126 CONNECTOR, P127 CONNECTOR, P128 CONNECTOR, P129 CONNECTOR, P13 BRANCH 2 BUS 1 LOAD 1 NO, P130 CONNECTOR, P131 CONNECTOR, P132 CONNECTOR, P133 CONNECTOR, P134 CONNECTOR, P135 CONNECTOR, P136 CONNECTOR, P137 CONNECTOR, P138 CONNECTOR, P139 CONNECTOR, P14 BRANCH 2 BUS 1 DISTAL NC, P140 CONNECTOR, P141 CONNECTOR, P142 CONNECTOR, P143 CONNECTOR, P144 CONNECTOR, P145 CONNECTOR, P146 CONNECTOR, P147 CONNECTOR, P148 CONNECTOR, P149 CONNECTOR, P15 BRANCH 2 BUS 1 DISTAL USER, P150 CONNECTOR, P151 CONNECTOR, P152 CONNECTOR, P153 CONNECTOR, P154 CONNECTOR, P155 CONNECTOR, P156 CONNECTOR, P157 CONNECTOR, P158 CONNECTOR, P159 CONNECTOR, P16 BRANCH 2 BUS 1 DISTAL NO, P160 CONNECTOR, P161 CONNECTOR, P162 CONNECTOR, P163 CONNECTOR, P164 CONNECTOR, P165 CONNECTOR, P166 CONNECTOR, P167 CONNECTOR, P168 CONNECTOR, P169 CONNECTOR, P17 BRANCH 2 BUS 1 PROXIMAL NC, P170 CONNECTOR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

Commit message: put power circuit on routing board
Parts:
- added D3: LED, ~, symbol LED
- added R4: 2.2k, ~, symbol R
- C2: renamed from C?; value C -> 1u
- C5: renamed from C?; value C -> 120u
- R1: renamed from R?; value R -> ctrl pulldown
- gave numbers to parts that had none: 16
Connections:
- net at C1.1, C2.1, C3.1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: now also D3.2 (K)
- net at F1.1, P302.1 (W): now also R4.2
- new net: D3.1 (A), R4.1
Changed lines of the file:
@@
 	41800 10100 41800 8450
 $Comp
-L PYB20 U?
+L PYB20 U1
 U 1 1 56F37FCD
 P 6050 27650
-F 0 "U?" H 6050 27650 60  0000 C CNN
+F 0 "U1" H 6050 27650 60  0000 C CNN
 F 1 "PYB20" H 6050 27750 60  0000 C CNN
 F 2 "~" H 6050 27650 60  0000 C CNN
@@
 $EndComp
 $Comp
-L CONNECTOR P?
+L CONNECTOR P302
 U 1 1 56F37FDC
 P 3450 27450
-F 0 "P?" H 3800 27550 70  0000 C CNN
+F 0 "P302" H 3800 27550 70  0000 C CNN
 F 1 "24Vin" H 3800 27350 70  0000 C CNN
 F 2 "~" H 3450 27450 60  0000 C CNN
@@
 $EndComp
 $Comp
-L CONNECTOR P?
+L CONNECTOR P303
 U 1 1 56F37FE9
 P 3450 28100
-F 0 "P?" H 3800 28200 70  0000 C CNN
+F 0 "P303" H 3800 28200 70  0000 C CNN
 F 1 "GND" H 3800 28000 70  0000 C CNN
 F 2 "~" H 3450 28100 60  0000 C CNN
@@
 $EndComp
 $Comp
-L CONNECTOR P?
+L CONNECTOR P304
 U 1 1 56F3854B
 P 7950 26700
-F 0 "P?" H 8300 26800 70  0000 C CNN
+F 0 "P304" H 8300 26800 70  0000 C CNN
 F 1 "+15V" H 8300 26600 70  0000 C CNN
 F 2 "~" H 7950 26700 60  0000 C CNN
@@
 $EndComp
 $Comp
-L CONNECTOR P?
+L CONNECTOR P305
 U 1 1 56F38551
 P 7950 28450
-F 0 "P?" H 8300 28550 70  0000 C CNN
+F 0 "P305" H 8300 28550 70  0000 C CNN
 F 1 "-15V" H 8300 28350 70  0000 C CNN
 F 2 "~" H 7950 28450 60  0000 C CNN
@@
 $EndComp
 $Comp
-L FUSE F?
+L FUSE F1
 U 1 1 56F38590
 P 3750 27450
-F 0 "F?" H 3850 27500 40  0000 C CNN
+F 0 "F1" H 3850 27500 40  0000 C CNN
 F 1 "FUSE" H 3650 27400 40  0000 C CNN
 F 2 "~" H 3750 27450 60  0000 C CNN
@@
 $EndComp
 $Comp
-L C C?
+L C C5
 U 1 1 56F3859F
 P 7200 27550
-F 0 "C?" H 7200 27650 40  0000 L CNN
-F 1 "C" H 7206 27465 40  0000 L CNN
+F 0 "C5" H 7200 27650 40  0000 L CNN
+F 1 "120u" H 7206 27465 40  0000 L CNN
 F 2 "~" H 7238 27400 30  0000 C CNN
 F 3 "~" H 7200 27550 60  0000 C CNN
@@
 $EndComp
 $Comp
-L INDUCTOR_SMALL L?
+L INDUCTOR_SMALL L1
 U 1 1 56F38CAF
 P 5000 27450
-F 0 "L?" H 5000 27550 50  0000 C CNN
+F 0 "L1" H 5000 27550 50  0000 C CNN
 F 1 "INDUCTOR_SMALL" H 5000 27400 50  0000 C CNN
 F 2 "~" H 5000 27450 60  0000 C CNN
@@
 $EndComp
 $Comp
-L C C?
+L C C4
 U 1 1 56F38CC8
 P 6050 26700
-F 0 "C?" H 6050 26800 40  0000 L CNN
+F 0 "C4" H 6050 26800 40  0000 L CNN
 F 1 "C" H 6056 26615 40  0000 L CNN
 F 2 "~" H 6088 26550 30  0000 C CNN
@@
 $EndComp
 $Comp
-L C C?
+L C C3
 U 1 1 56F38CD5
 P 6000 28450
-F 0 "C?" H 6000 28550 40  0000 L CNN
+F 0 "C3" H 6000 28550 40  0000 L CNN
 F 1 "C" H 6006 28365 40  0000 L CNN
 F 2 "~" H 6038 28300 30  0000 C CNN
@@
 $EndComp
 $Comp
-L C C?
+L C C2
 U 1 1 56F38CDB
 P 4600 27800
-F 0 "C?" H 4600 27900 40  0000 L CNN
-F 1 "C" H 4606 27715 40  0000 L CNN
+F 0 "C2" H 4600 27900 40  0000 L CNN
+F 1 "1u" H 4606 27715 40  0000 L CNN
 F 2 "~" H 4638 27650 30  0000 C CNN
 F 3 "~" H 4600 27800 60  0000 C CNN
@@
 $EndComp
 $Comp
-L C C?
+L C C1
 U 1 1 56F38CE1
 P 4350 27800
-F 0 "C?" H 4350 27900 40  0000 L CNN
+F 0 "C1" H 4350 27900 40  0000 L CNN
 F 1 "330u" H 4356 27715 40  0000 L CNN
 F 2 "~" H 4388 27650 30  0000 C CNN
@@
 $EndComp
 $Comp
-L VR VR?
+L VR VR1
 U 1 1 56F38CF8
 P 4100 27800
-F 0 "VR?" V 4160 27754 40  0000 C TNN
+F 0 "VR1" V 4160 27754 40  0000 C TNN
 F 1 "VR" V 4100 27800 40  0000 C CNN
 F 2 "~" H 4100 27800 60  0000 C CNN
@@
 Connection ~ 7200 28450
 $Comp
-L R R?
+L R R2
 U 1 1 56F3B8F8
 P 7850 27000
-F 0 "R?" V 7930 27000 40  0000 C CNN
+F 0 "R2" V 7930 27000 40  0000 C CNN
 F 1 "2.2k" V 7857 27001 40  0000 C CNN
 F 2 "~" V 7780 27000 30  0000 C CNN
@@
 $EndComp
 $Comp
-L R R?
+L R R3
 U 1 1 56F3B905
 P 7850 28150
-F 0 "R?" V 7930 28150 40  0000 C CNN
+F 0 "R3" V 7930 28150 40  0000 C CNN
 F 1 "2.2k" V 7857 28151 40  0000 C CNN
 F 2 "~" V 7780 28150 30  0000 C CNN
@@
 $EndComp
 $Comp
-L LED D?
+L LED D1
 U 1 1 56F3B90D
 P 7600 27350
-F 0 "D?" H 7600 27450 50  0000 C CNN
+F 0 "D1" H 7600 27450 50  0000 C CNN
 F 1 "LED" H 7600 27250 50  0000 C CNN
 F 2 "~" H 7600 27350 60  0000 C CNN
@@
 $EndComp
 $Comp
-L LED D?
+L LED D2
 U 1 1 56F3B92E
 P 7600 27550
-F 0 "D?" H 7600 27650 50  0000 C CNN
+F 0 "D2" H 7600 27650 50  0000 C CNN
 F 1 "LED" H 7600 27450 50  0000 C CNN
 F 2 "~" H 7600 27550 60  0000 C CNN
@@
 Connection ~ 7850 28450
 $Comp
-L SPST SW?
+L SPST SW1
 U 1 1 56F3C6DF
 P 4650 28450
-F 0 "SW?" H 4650 28550 70  0000 C CNN
+F 0 "SW1" H 4650 28550 70  0000 C CNN
 F 1 "SPST" H 4650 28350 70  0000 C CNN
 F 2 "~" H 4650 28450 60  0000 C CNN
@@
 Connection ~ 4100 28100
 $Comp
-L R R?
+L R R1
 U 1 1 56F3CCA3
 P 3800 28450
-F 0 "R?" V 3880 28450 40  0000 C CNN
-F 1 "R" V 3807 28451 40  0000 C CNN
+F 0 "R1" V 3880 28450 40  0000 C CNN
+F 1 "ctrl pulldown" V 3807 28451 40  0000 C CNN
 F 2 "~" V 3730 28450 30  0000 C CNN
 F 3 "~" H 3800 28450 30  0000 C CNN
@@
 $EndComp
 Wire Wire Line
-	3550 28450 3500 28450
-Wire Wire Line
-	3500 28450 3500 28100
+	3500 28450 3550 28450
+Wire Wire Line
+	3500 27850 3500 28450
 Connection ~ 3500 28100
 Wire Wire Line
 	4050 28450 4150 28450
+$Comp
+L R R4
+U 1 1 56F3D170
+P 2600 27650
+F 0 "R4" V 2680 27650 40  0000 C CNN
+F 1 "2.2k" V 2607 27651 40  0000 C CNN
+F 2 "~" V 2530 27650 30  0000 C CNN
+F 3 "~" H 2600 27650 30  0000 C CNN
+	1    2600 27650
+	0    -1   -1   0
+$EndComp
+$Comp
+L LED D3
+U 1 1 56F3D17D
+P 2600 27850
+F 0 "D3" H 2600 27950 50  0000 C CNN
+F 1 "LED" H 2600 27750 50  0000 C CNN
+F 2 "~" H 2600 27850 60  0000 C CNN
+F 3 "~" H 2600 27850 60  0000 C CNN
+	1    2600 27850
+	1    0    0    -1
+$EndComp
+Wire Wire Line
+	2850 27650 3500 27650
+Wire Wire Line
+	3500 27650 3500 27450
+Wire Wire Line
+	2350 27650 2300 27650
+Wire Wire Line
+	2300 27650 2300 27850
+Wire Wire Line
+	2300 27850 2400 27850
+Wire Wire Line
+	2800 27850 3500 27850
 $EndSCHEMATC
