File: DCMGv2SOURCEStest.sch (KiCad schematic (older format))
At the start: 154 parts, among them P10 NC_SCGR_SIG, P14 UNREG_V_SIG, P15 UNREG_I_SIG, P16 TO_REG+, P17 TO_REG-, P18 FROM_REG+, P19 FROM_REG-, P20 REG_V_SIG, P21 TO_GRID-, P22 REG_I_SIG, P23 TO_GRID+, P3 FROM_SRC+, P4 CTRL_SIG, P5 FROM_SRC-, P6 GND_IN, P7 IC+IN, P8 IC-IN, P9 COIL+IN, Q1 STS1DNC45, Q2 IRFP260, Q3 STS1DNC45, Q4 IRF5210, Q5 IRF5210, SW1 SPDT_RELAY, SW2 SPDT_RELAY, U1 LT1014DN, U10 LT1634, U11 LT1010, U12 LT1014DN, U13 LT1014DN, U14 ULN2803A, U2 LM339, U3 LT1634, U6 DAUGHTERBOARD_MOUNT, U7 LT1014DN, U8 LT1014DN, U9 LT1014DN

Commit message: added power indicators. added mounting holes. board size increased slightly in y dim. fixed important schematic and routing error involving U8B and U8D!
Parts:
- added D11, D12, D2: LED_RED, ~, symbol LED
- added R10, R6, R7: 2.2k, ~, symbol R
Connections:
- wire segments 404 -> 412
Other:
- moved on the sheet: C6, C7, C8, P7, P8, P9

Commit message: replaced SPST slider footprint. More importantly, I fixed the following issues from the prototype test source board: 1. over current protection transistor drain and source were reversed. 2. U12 negative supply disconnected. 3. screw terminals inaccessible with daughterboard in place. 4. lack of reverse bias protection.
Parts:
- added D13, D14, D16: DIODESCH, ~, symbol DIODESCH
Connections:
- wire segments 412 -> 422
Other:
- moved on the sheet: P7, P8, P9
Changed lines of the file:
@@
 Sheet 1 1
 Title ""
-Date "3 mar 2016"
+Date "31 mar 2016"
 Rev ""
 Comp ""
@@
 L CONNECTOR P7
 U 1 1 56094E47
-P 5450 1650
-F 0 "P7" H 5800 1750 70  0000 C CNN
-F 1 "IC+IN" H 5800 1550 70  0000 C CNN
-F 2 "~" H 5450 1650 60  0000 C CNN
-F 3 "~" H 5450 1650 60  0000 C CNN
-	1    5450 1650
+P 4900 1650
+F 0 "P7" H 5250 1750 70  0000 C CNN
+F 1 "IC+IN" H 5250 1550 70  0000 C CNN
+F 2 "~" H 4900 1650 60  0000 C CNN
+F 3 "~" H 4900 1650 60  0000 C CNN
+	1    4900 1650
 	-1   0    0    1
 $EndComp
@@
 L CONNECTOR P8
 U 1 1 56094E48
-P 5400 4150
-F 0 "P8" H 5750 4250 70  0000 C CNN
-F 1 "IC-IN" H 5750 4050 70  0000 C CNN
-F 2 "~" H 5400 4150 60  0000 C CNN
-F 3 "~" H 5400 4150 60  0000 C CNN
-	1    5400 4150
+P 4900 4150
+F 0 "P8" H 5250 4250 70  0000 C CNN
+F 1 "IC-IN" H 5250 4050 70  0000 C CNN
+F 2 "~" H 4900 4150 60  0000 C CNN
+F 3 "~" H 4900 4150 60  0000 C CNN
+	1    4900 4150
 	-1   0    0    1
 $EndComp
@@
 L CONNECTOR P9
 U 1 1 56094E4B
-P 6650 1750
-F 0 "P9" H 7000 1850 70  0000 C CNN
-F 1 "COIL+IN" H 7000 1650 70  0000 C CNN
-F 2 "~" H 6650 1750 60  0000 C CNN
-F 3 "~" H 6650 1750 60  0000 C CNN
-	1    6650 1750
+P 6350 1750
+F 0 "P9" H 6700 1850 70  0000 C CNN
+F 1 "COIL+IN" H 6700 1650 70  0000 C CNN
+F 2 "~" H 6350 1750 60  0000 C CNN
+F 3 "~" H 6350 1750 60  0000 C CNN
+	1    6350 1750
 	-1   0    0    1
 $EndComp
@@
 Connection ~ 5500 1650
 Wire Wire Line
-	5500 1700 5500 1650
+	5500 1650 5500 1700
 Wire Wire Line
 	5500 2250 5500 2100
@@
 Connection ~ 5500 4150
 Wire Wire Line
-	5500 4050 5500 4150
+	5500 4150 5500 4050
 Connection ~ 5050 2900
 Wire Wire Line
@@
 Connection ~ 8250 9050
 Wire Wire Line
-	8250 9150 8250 9050
+	8250 9050 8250 9150
 Connection ~ 8250 9600
 Wire Wire Line
@@
 	9600 13950 9550 13950
 Wire Wire Line
-	9550 14000 9550 13900
+	9550 13900 9550 14000
 Connection ~ 9550 13350
 Connection ~ 12150 12650
@@
 	12100 12650 12150 12650
 Wire Wire Line
-	12150 12700 12150 12600
+	12150 12600 12150 12700
 Connection ~ 15600 5050
 Wire Wire Line
@@
 Connection ~ 5450 9150
 Wire Wire Line
-	5450 9550 5450 9150
+	5450 9150 5450 9550
 Wire Wire Line
-	5600 9550 5450 9550
+	5450 9550 5600 9550
 Connection ~ 4650 9150
 Wire Wire Line
@@
 Connection ~ 5100 9750
 Wire Wire Line
-	5100 9850 5100 9750
+	5100 9550 5100 9850
 Wire Wire Line
 	7500 7250 7500 9950
@@
 	5400 12800 5500 12800
 Wire Wire Line
-	5500 13350 5500 11500
+	5500 11500 5500 13350
 Wire Wire Line
-	4550 13350 5500 13350
+	5500 13350 4550 13350
 Wire Wire Line
-	4550 12950 4550 13350
+	4550 13350 4550 12950
 Wire Wire Line
-	4600 12950 4550 12950
+	4550 12950 4600 12950
 Connection ~ 4350 12650
 Wire Wire Line
@@
 	5500 11500 5200 11500
 Wire Wire Line
-	18750 5600 18750 12250
+	18750 12250 18750 5600
 Wire Wire Line
 	17900 8850 17900 8550
@@
 	17550 5600 17550 5750
 Wire Wire Line
-	17550 5600 18750 5600
+	18750 5600 17550 5600
 Wire Wire Line
 	18050 5750 18050 5600
@@
 Connection ~ 6700 9750
 Wire Wire Line
-	6700 10850 6700 9750
+	6700 9750 6700 10850
 Wire Wire Line
 	5800 10650 5800 10850
@@
 	9500 10300 9500 9750
 Wire Wire Line
-	8700 10000 8700 9750
+	8700 9750 8700 10000
 Wire Wire Line
 	10550 10400 10550 11400
@@
 Connection ~ 7700 9750
 Wire Wire Line
-	7700 9950 7700 9750
+	7700 9750 7700 9950
 Wire Wire Line
 	7700 10650 7700 10450
@@
 Connection ~ 8850 9050
 Wire Wire Line
-	8850 9100 8850 9050
+	8850 9050 8850 9100
 Wire Wire Line
 	8850 9600 8850 9500
@@
 Connection ~ 12700 4950
 Wire Wire Line
-	12700 4900 12700 4950
+	12700 4950 12700 4900
 Connection ~ 12950 4950
 Wire Wire Line
-	12950 4900 12950 4950
+	12950 4950 12950 4900
 Connection ~ 13200 4950
 Wire Wire Line
-	13200 4900 13200 4950
+	13200 4950 13200 4900
 Wire Wire Line
 	13450 4950 13450 4900
 Connection ~ 12700 4450
 Wire Wire Line
-	12700 4500 12700 4450
+	12700 4450 12700 4500
 Connection ~ 12950 4450
 Wire Wire Line
-	12950 4500 12950 4450
+	12950 4450 12950 4500
 Connection ~ 13200 4450
 Wire Wire Line
-	13200 4500 13200 4450
+	13200 4450 13200 4500
 Wire Wire Line
 	13450 4450 13450 4500
 Connection ~ 11450 4450
 Wire Wire Line
-	11450 4500 11450 4450
+	11450 4450 11450 4500
 Connection ~ 11200 4450
 Wire Wire Line
-	11200 4500 11200 4450
+	11200 4450 11200 4500
 Connection ~ 10950 4450
 Wire Wire Line
@@
 Connection ~ 11450 4950
 Wire Wire Line
-	11450 4900 11450 4950
+	11450 4950 11450 4900
 Connection ~ 11200 4950
 Wire Wire Line
-	11200 4900 11200 4950
+	11200 4950 11200 4900
 Connection ~ 10950 4950
 Wire Wire Line
@@
 Connection ~ 11400 5650
 Wire Wire Line
-	11400 5700 11400 5650
+	11400 5650 11400 5700
 Connection ~ 11150 5650
 Wire Wire Line
-	11150 5700 11150 5650
+	11150 5650 11150 5700
 Connection ~ 10900 5650
 Wire Wire Line
@@
 Connection ~ 11400 6150
 Wire Wire Line
-	11400 6100 11400 6150
+	11400 6150 11400 6100
 Connection ~ 11150 6150
 Wire Wire Line
-	11150 6100 11150 6150
+	11150 6150 11150 6100
 Connection ~ 10900 6150
 Wire Wire Line
@@
 Connection ~ 12800 6150
 Wire Wire Line
-	12800 6100 12800 6150
+	12800 6150 12800 6100
 Connection ~ 13050 6150
 Wire Wire Line
-	13050 6100 13050 6150
+	13050 6150 13050 6100
 Connection ~ 13300 6150
 Wire Wire Line
-	13300 6100 13300 6150
+	13300 6150 13300 6100
 Connection ~ 12550 6150
 Wire Wire Line
@@
 Connection ~ 12800 5650
 Wire Wire Line
-	12800 5700 12800 5650
+	12800 5650 12800 5700
 Connection ~ 13050 5650
 Wire Wire Line
-	13050 5700 13050 5650
+	13050 5650 13050 5700
 Connection ~ 13300 5650
 Wire Wire Line
-	13300 5700 13300 5650
+	13300 5650 13300 5700
 Connection ~ 12550 5650
 Wire Wire Line
@@
 	13150 12250 14900 12250
 Wire Wire Line
-	18750 12250 15400 12250
+	15400 12250 18750 12250
 Connection ~ 14250 9900
 Wire Wire Line
-	14150 9900 14250 9900
+	14250 9900 14150 9900
 Connection ~ 13650 9750
 Wire Wire Line
-	13650 9900 13650 9750
+	13650 9750 13650 9900
 Wire Wire Line
-	13750 9900 13650 9900
+	13650 9900 13750 9900
 Connection ~ 11250 9750
 Wire Wire Line
@@
 	14600 8500 14850 8500
 Wire Wire Line
-	14600 9050 14600 9000
-Wire Wire Line
-	14450 9050 14600 9050
-Wire Wire Line
 	15050 8550 15050 9050
 Wire Wire Line
-	15950 8550 15950 9050
+	15950 9050 15950 8550
 Wire Wire Line
 	15200 5750 15200 5650
@@
 	15150 10100 14900 10100
 Wire Wire Line
-	13200 9050 14050 9050
-Wire Wire Line
 	12400 12100 12400 12200
 Wire Wire Line
@@
 Connection ~ 12000 9750
 Wire Wire Line
-	5600 1650 5450 1650
+	4900 1650 5600 1650
 Wire Wire Line
-	5400 4150 5550 4150
+	4900 4150 5550 4150
 Wire Wire Line
 	12300 10750 12100 10750
@@
 Connection ~ 12300 9050
 Wire Wire Line
-	6650 1750 6800 1750
+	6350 1750 6800 1750
 Connection ~ 11550 9750
 Wire Wire Line
@@
 Wire Wire Line
 	10050 11250 10050 11650
+Wire Wire Line
+	13200 9050 14000 9050
+Wire Wire Line
+	14000 9050 14000 8950
+Wire Wire Line
+	14000 8950 14500 8950
+Wire Wire Line
+	14500 8950 14500 9050
+Wire Wire Line
+	14500 9050 14450 9050
+Wire Wire Line
+	14600 9000 14050 9000
+Wire Wire Line
+	14050 9000 14050 9050
+$Comp
+L DIODESCH D13
+U 1 1 56FCAE5B
+P 5150 2250
+F 0 "D13" H 5150 2350 40  0000 C CNN
+F 1 "DIODESCH" H 5150 2150 40  0000 C CNN
+F 2 "~" H 5150 2250 60  0000 C CNN
+F 3 "~" H 5150 2250 60  0000 C CNN
+	1    5150 2250
+	0    -1   -1   0
+$EndComp
+$Comp
+L DIODESCH D14
+U 1 1 56FCAE68
+P 5150 3500
+F 0 "D14" H 5150 3600 40  0000 C CNN
+F 1 "DIODESCH" H 5150 3400 40  0000 C CNN
+F 2 "~" H 5150 3500 60  0000 C CNN
+F 3 "~" H 5150 3500 60  0000 C CNN
+	1    5150 3500
+	0    -1   -1   0
+$EndComp
+Wire Wire Line
+	5150 2450 5150 3300
+Connection ~ 5150 2900
+Wire Wire Line
+	5150 2050 5150 1650
+Connection ~ 5150 1650
+Wire Wire Line
+	5150 3700 5150 4150
+Connection ~ 5150 4150
+Connection ~ 6450 1750
+$Comp
+L DIODESCH D16
+U 1 1 56FCBE85
+P 3450 9550
+F 0 "D16" H 3450 9650 40  0000 C CNN
+F 1 "DIODESCH" H 3450 9450 40  0000 C CNN
+F 2 "~" H 3450 9550 60  0000 C CNN
+F 3 "~" H 3450 9550 60  0000 C CNN
+	1    3450 9550
+	-1   0    0    1
+$EndComp
+Wire Wire Line
+	3250 9550 3000 9550
+Wire Wire Line
+	3000 9550 3000 9050
+Connection ~ 3000 9050
+Wire Wire Line
+	3650 9550 5100 9550
 $EndSCHEMATC
