File: DCMGv2SOURCEStest.sch (KiCad schematic (older format))
At the start: 165 parts, among them P10 NC_SCGR_SIG, P14 UNREG_V_SIG, P15 UNREG_I_SIG, P16 TO_REG+, P17 TO_REG-, P18 FROM_REG+, P19 FROM_REG-, P20 REG_V_SIG, P21 TO_GRID-, P22 REG_I_SIG, P23 TO_GRID+, P3 FROM_SRC+, P4 CTRL_SIG, P5 FROM_SRC-, P6 GND_IN, P7 IC+IN, P8 IC-IN, P9 COIL+IN, Q1 STS1DNC45, Q2 IRFP260, Q3 STS1DNC45, Q4 IRF5210, Q5 IRF5210, SW1 SPDT_RELAY, SW2 SPDT_RELAY, U1 LT1014DN, U10 LT1634, U11 LT1010, U12 LT1014DN, U13 LT1014DN, U14 ULN2803A, U2 LM339, U3 LT1634, U6 DAUGHTERBOARD_MOUNT, U7 LT1014DN, U8 LT1014DN, U9 LT1014DN

Commit message: added optional filtering capacitors for measurement amplifiers. corrected zener clamps to clamp high AND low voltages.
Parts:
- added C3, C4, C5, C9, C?: C, ~, symbol C
- added D15, D17, D18, D19: BZX84C10L, ~, symbol ZENER
Connections:
- wire segments 435 -> 455

Commit message: separated transistors for heat sink clearance
Parts:
- added R12: 10M, ~, symbol R
- C1, C2: value C -> 10n
- C10: renamed from C?; value C -> 2.2n
- C3, C4, C5, C9: value C -> 2.2n
Connections:
- wire segments 455 -> 457
Changed lines of the file:
@@
 Sheet 1 1
 Title ""
-Date "9 apr 2016"
+Date "11 apr 2016"
 Rev ""
 Comp ""
@@
 P 11100 10000
 F 0 "C2" H 11100 10100 40  0000 L CNN
-F 1 "C" H 11106 9915 40  0000 L CNN
+F 1 "10n" H 11106 9915 40  0000 L CNN
 F 2 "~" H 11138 9850 30  0000 C CNN
 F 3 "~" H 11100 10000 60  0000 C CNN
@@
 P 9100 9950
 F 0 "C1" H 9100 10050 40  0000 L CNN
-F 1 "C" H 9106 9865 40  0000 L CNN
+F 1 "10n" H 9106 9865 40  0000 L CNN
 F 2 "~" H 9138 9800 30  0000 C CNN
 F 3 "~" H 9100 9950 60  0000 C CNN
@@
 	13150 12150 13150 11900
 Connection ~ 15650 12250
-Connection ~ 13150 12150
 Wire Wire Line
 	15650 12150 13150 12150
@@
 Wire Wire Line
 	3400 8700 3400 8500
-Connection ~ 13150 12250
 Wire Wire Line
 	13000 10000 13000 10200
@@
 Connection ~ 13000 10050
 Wire Wire Line
-	12500 10050 13000 10050
+	12500 10050 13600 10050
 Wire Wire Line
 	12500 10250 12500 10050
@@
 	13400 11350 13400 11400
 Wire Wire Line
-	13150 11350 13400 11350
+	13150 11350 13600 11350
 Wire Wire Line
 	13150 11000 13150 11400
@@
 Wire Wire Line
 	6350 1750 6800 1750
-Connection ~ 11550 9750
 Wire Wire Line
 	11950 4450 11950 4500
@@
 P 9050 13650
 F 0 "C3" H 9050 13750 40  0000 L CNN
-F 1 "C" H 9056 13565 40  0000 L CNN
+F 1 "2.2n" H 9056 13565 40  0000 L CNN
 F 2 "~" H 9088 13500 30  0000 C CNN
 F 3 "~" H 9050 13650 60  0000 C CNN
@@
 P 10300 12950
 F 0 "C4" H 10300 13050 40  0000 L CNN
-F 1 "C" H 10306 12865 40  0000 L CNN
+F 1 "2.2n" H 10306 12865 40  0000 L CNN
 F 2 "~" H 10338 12800 30  0000 C CNN
 F 3 "~" H 10300 12950 60  0000 C CNN
@@
 P 11350 11450
 F 0 "C5" H 11350 11550 40  0000 L CNN
-F 1 "C" H 11356 11365 40  0000 L CNN
+F 1 "2.2n" H 11356 11365 40  0000 L CNN
 F 2 "~" H 11388 11300 30  0000 C CNN
 F 3 "~" H 11350 11450 60  0000 C CNN
@@
 P 16350 6000
 F 0 "C9" H 16350 6100 40  0000 L CNN
-F 1 "C" H 16356 5915 40  0000 L CNN
+F 1 "2.2n" H 16356 5915 40  0000 L CNN
 F 2 "~" H 16388 5850 30  0000 C CNN
 F 3 "~" H 16350 6000 60  0000 C CNN
@@
 Connection ~ 8900 13200
 $Comp
-L C C?
+L C C10
 U 1 1 5708F0A5
 P 18300 5950
-F 0 "C?" H 18300 6050 40  0000 L CNN
-F 1 "C" H 18306 5865 40  0000 L CNN
+F 0 "C10" H 18300 6050 40  0000 L CNN
+F 1 "2.2n" H 18306 5865 40  0000 L CNN
 F 2 "~" H 18338 5800 30  0000 C CNN
 F 3 "~" H 18300 5950 60  0000 C CNN
@@
 	18300 6400 18050 6400
 Connection ~ 18050 6400
+$Comp
+L R R12
+U 1 1 570AF8AC
+P 13600 10800
+F 0 "R12" V 13680 10800 40  0000 C CNN
+F 1 "10M" V 13607 10801 40  0000 C CNN
+F 2 "~" V 13530 10800 30  0000 C CNN
+F 3 "~" H 13600 10800 30  0000 C CNN
+	1    13600 10800
+	1    0    0    -1
+$EndComp
+Wire Wire Line
+	13600 10050 13600 10550
+Wire Wire Line
+	13600 11350 13600 11050
+Connection ~ 13400 11350
 $EndSCHEMATC
