File: DCMGv2_SIGNALROUTING.kicad_pcb (KiCad board)
At the start: 2 copper layers, 258.1 x 163.1 mm, 333 parts, among them P1 BRANCH 1 BUS 1 LOAD3 NC, P10 BRANCH 1 BUS 1 LOAD 2 NC, P100 CONNECTOR, P101 CONNECTOR, P102 CONNECTOR, P103 CONNECTOR, P104 CONNECTOR, P105 CONNECTOR, P106 CONNECTOR, P107 CONNECTOR, P108 CONNECTOR, P109 CONNECTOR, P11 BRANCH 1 BUS 1 LOAD 1 NO, P110 CONNECTOR, P111 CONNECTOR, P112 CONNECTOR, P113 CONNECTOR, P114 CONNECTOR, P115 CONNECTOR, P116 CONNECTOR, P117 CONNECTOR, P118 CONNECTOR, P119 CONNECTOR, P12 BRANCH 1 BUS 1 LOAD 1 NC, P120 CONNECTOR, P121 CONNECTOR, P122 CONNECTOR, P123 CONNECTOR, P124 CONNECTOR, P125 CONNECTOR, P126 CONNECTOR, P127 CONNECTOR, P128 CONNECTOR, P129 CONNECTOR, P13 BRANCH 2 BUS 1 LOAD 1 NO, P130 CONNECTOR, P131 CONNECTOR, P132 CONNECTOR, P133 CONNECTOR, P134 CONNECTOR, P135 CONNECTOR, P136 CONNECTOR, P137 CONNECTOR, P138 CONNECTOR, P139 CONNECTOR, P14 BRANCH 2 BUS 1 DISTAL NC, P140 CONNECTOR, P141 CONNECTOR, P142 CONNECTOR, P143 CONNECTOR, P144 CONNECTOR, P145 CONNECTOR, P146 CONNECTOR, P147 CONNECTOR, P148 CONNECTOR, P149 CONNECTOR, P15 BRANCH 2 BUS 1 DISTAL USER, P150 CONNECTOR, P151 CONNECTOR, P152 CONNECTOR, P153 CONNECTOR, P154 CONNECTOR, P155 CONNECTOR, P156 CONNECTOR, P157 CONNECTOR, P158 CONNECTOR, P159 CONNECTOR, P16 BRANCH 2 BUS 1 DISTAL NO, P160 CONNECTOR, P161 CONNECTOR, P162 CONNECTOR, P163 CONNECTOR, P164 CONNECTOR, P165 CONNECTOR, P166 CONNECTOR, P167 CONNECTOR, P168 CONNECTOR, P169 CONNECTOR, P17 BRANCH 2 BUS 1 PROXIMAL NC, P170 CONNECTOR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

Commit message: replaced SPST slider footprint. More importantly, I fixed the following issues from the prototype test source board: 1. over current protection transistor drain and source were reversed. 2. U12 negative supply disconnected. 3. screw terminals inaccessible with daughterboard in place. 4. lack of reverse bias protection.
Changed lines of the file:
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@@
     (links 189)
     (no_connects 8)
-    (area 50.182857 61.746 309.499 231.069444)
+    (area 50.749999 61.925999 308.914001 225.094001)
     (thickness 1.6)
     (drawings 66)
@@
     )
   )
-  (module L101011MS02_SPDT (layer F.Cu)
-    (at 194.564 220.472)
-    (fp_text reference SW1 (at 0 -3.556) (layer F.SilkS)
-      (effects (font (size 1 1) (thickness 0.15)))
-    )
-    (fp_text value SPST (at 0 -1.778) (layer F.SilkS)
-      (effects (font (size 1 1) (thickness 0.15)))
-    )
-    (fp_line (start 9.55 -8.25) (end -9.55 -8.25) (layer F.SilkS) (width 0.3))
-    (fp_line (start -9.55 -8.25) (end -9.55 2.54) (layer F.SilkS) (width 0.3))
-    (fp_line (start -9.55 2.54) (end 9.55 2.54) (layer F.SilkS) (width 0.3))
-    (fp_line (start 9.55 -8.25) (end 9.55 2.54) (layer F.SilkS) (width 0.3))
-    (pad 1 thru_hole oval (at -4.6 -5.7) (size 1.52 0.762) (drill oval 1.27 0.51)
-      (layers *.Cu *.Mask F.SilkS)
-      (net 129 N-0000073)
-    )
-    (pad 2 thru_hole oval (at 0 -5.7) (size 1.52 0.762) (drill oval 1.27 0.51)
-      (layers *.Cu *.Mask F.SilkS)
-      (net 132 N-0000076)
-    )
-    (pad 3 thru_hole oval (at 4.6 -5.7) (size 1.52 0.762) (drill oval 1.27 0.51)
-      (layers *.Cu *.Mask F.SilkS)
-    )
-    (pad 4 thru_hole oval (at -4.6 0) (size 1.52 0.762) (drill oval 1.27 0.51)
-      (layers *.Cu *.Mask F.SilkS)
-    )
-    (pad 5 thru_hole oval (at 0 0) (size 1.52 0.762) (drill oval 1.27 0.51)
-      (layers *.Cu *.Mask F.SilkS)
-    )
-    (pad 6 thru_hole oval (at 4.6 0) (size 1.52 0.762) (drill oval 1.27 0.51)
-      (layers *.Cu *.Mask F.SilkS)
-    )
-  )
   (module FR-A_50v (layer F.Cu)
     (at 108.966 197.612 90)
@@
       (layers *.Cu *.Mask F.SilkS)
     )
+  )
+  (module L101011MS02_SPDT (layer F.Cu)
+    (at 194.564 220.472)
+    (fp_text reference SW1 (at 0 -3.556) (layer F.SilkS)
+      (effects (font (size 1 1) (thickness 0.15)))
+    )
+    (fp_text value SPST (at 0 -1.778) (layer F.SilkS)
+      (effects (font (size 1 1) (thickness 0.15)))
+    )
+    (fp_line (start 9.55 -8.25) (end -9.55 -8.25) (layer F.SilkS) (width 0.3))
+    (fp_line (start -9.55 -8.25) (end -9.55 2.54) (layer F.SilkS) (width 0.3))
+    (fp_line (start -9.55 2.54) (end 9.55 2.54) (layer F.SilkS) (width 0.3))
+    (fp_line (start 9.55 -8.25) (end 9.55 2.54) (layer F.SilkS) (width 0.3))
+    (pad 1 thru_hole circle (at -4.6 -5.7) (size 1.52 1.52) (drill 1.27)
+      (layers *.Cu *.Mask F.SilkS)
+      (net 129 N-0000073)
+    )
+    (pad 2 thru_hole circle (at 0 -5.7) (size 1.52 1.52) (drill 1.27)
+      (layers *.Cu *.Mask F.SilkS)
+      (net 132 N-0000076)
+    )
+    (pad 3 thru_hole circle (at 4.6 -5.7) (size 1.52 1.52) (drill 1.27)
+      (layers *.Cu *.Mask F.SilkS)
+    )
+    (pad 4 thru_hole circle (at -4.6 0) (size 1.52 1.52) (drill 1.27)
+      (layers *.Cu *.Mask F.SilkS)
+    )
+    (pad 5 thru_hole circle (at 0 0) (size 1.52 1.52) (drill 1.27)
+      (layers *.Cu *.Mask F.SilkS)
+    )
+    (pad 6 thru_hole circle (at 4.6 0) (size 1.52 1.52) (drill 1.27)
+      (layers *.Cu *.Mask F.SilkS)
+    )
