File: DCMGv2SOURCES.kicad_pcb (KiCad board)
At the start: 2 copper layers, 253 x 74.2 mm, 165 parts, among them P10 NC_SCGR_SIG, P14 UNREG_V_SIG, P15 UNREG_I_SIG, P16 TO_REG+, P17 TO_REG-, P18 FROM_REG+, P19 FROM_REG-, P20 REG_V_SIG, P21 TO_GRID-, P22 REG_I_SIG, P23 TO_GRID+, P3 FROM_SRC+, P4 CTRL_SIG, P5 FROM_SRC-, P6 GND_IN, P7 IC+IN, P8 IC-IN, P9 COIL+IN, Q1 STS1DNC45, Q2 IRFP260, Q3 STS1DNC45, Q4 IRF5210, Q5 IRF5210, SW1 SPDT_RELAY, SW2 SPDT_RELAY, U1 LT1014DN, U10 LT1634, U11 LT1010, U12 LT1014DN, U13 LT1014DN, U14 ULN2803A, U2 LM339, U3 LT1634, U6 DAUGHTERBOARD_MOUNT, U7 LT1014DN, U8 LT1014DN, U9 LT1014DN

Commit message: replaced SPST slider footprint. More importantly, I fixed the following issues from the prototype test source board: 1. over current protection transistor drain and source were reversed. 2. U12 negative supply disconnected. 3. screw terminals inaccessible with daughterboard in place. 4. lack of reverse bias protection.
Parts:
- added 3mm_hole: VAL**, 3mm_hole, F.Cu at (102.6, 21.8)
- added 3mm_hole: VAL**, 3mm_hole, F.Cu at (48.5, 81.8)
- added D13: DIODESCH, R6, F.Cu at (52.3, 85.9)
- added D14: DIODESCH, R6, F.Cu at (33.3, 85.9)
- added D16: DIODESCH, R6, B.Cu at (80.8, 28.7)
- moved P10 70.1 mm to (121.2, 86.4)
- moved P4 65.0 mm to (118.6, 86.4)
- moved D2 55.1 mm to (97.3, 86.1)
- moved R6 54.1 mm to (92.2, 86.1), turned to 0 degrees
- moved D11 50.5 mm to (79.0, 86.4), turned to 180 degrees
- moved R7 41.1 mm to (73.9, 86.4), turned to 180 degrees
- moved P19 37.5 mm to (225.8, 75.7)
- moved 3mm_hole 31.7 mm to (45.2, 20.1)
- moved 3mm_hole 25.3 mm to (143.0, 83.3)
- moved R64 23.6 mm to (220.7, 32.8), turned to 0 degrees
- moved 3mm_hole 20.6 mm to (241.3, 83.8)
- moved 3mm_hole 20.6 mm to (241.3, 20.3)
- moved P23 17.8 mm to (232.4, 40.1)
- moved R62 17.4 mm to (234.2, 49.5), turned to 180 degrees
- moved P21 16.9 mm to (232.4, 59.4)
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Connections:
- Q4 pad 1: N-0000050 (its old number) -> N-0000054
- Q5 pad 1: N-0000052 (its old number) -> N-0000054
- Q5 pad 3: N-0000050 (its old number) -> N-0000053
- R57 pad 2: N-0000052 (its old number) -> N-0000053
Routing:
- net N-0000027: track 75.9 -> 4.78 mm
- net N-0000029: track 69.5 -> 4.89 mm
- net IC_POW-: track 311.6 -> 362.8 mm, vias 13 -> 16
- net N-0000052 (its old number): track 32.7 -> 0.00 mm
- net N-0000042: track 157.0 -> 125.1 mm
- net N-0000053: track 0.00 -> 23.7 mm
- net N-0000054: track 0.00 -> 22.1 mm
- net N-0000050 (its old number): track 20.0 -> 0.00 mm
- net N-0000085: track 125.5 -> 139.2 mm
- net N-0000065: track 158.5 -> 147.7 mm
- net N-0000026: track 57.2 -> 62.2 mm
- net CTRL_GND: track 156.6 -> 158.7 mm
- net COIL_POW+: track 207.5 -> 209.5 mm
- net N-0000055: track 54.8 -> 56.6 mm
- net N-0000056: track 47.5 -> 49.3 mm
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Other:
- board size 253 x 74.2 mm -> 236.5 x 74.2 mm
- board text added: "IC+"
- board text added: "IC-"
- board text added: "SINGLE CH SOURCE BOARD v1.1 JORDAN MURRAY jmm72@case.edu MAR 2016"
- board text removed: "SINGLE CH SOURCE BOARD v1.0 JORDAN MURRAY - jmm72@case.edu MAR 2016"

Commit message: reduce need for output voltage protection by switching output current sensing to low side. made associated changes in output voltage measurement (Vout+ to Vout- is now distinct from Vout+ to gnd)
Parts:
- moved C25 64.6 mm to (230.4, 28.2), turned to 180 degrees
- moved R64 41.8 mm to (230.4, 73.4)
- moved P19 8.59 mm to (217.7, 78.5)
- moved P21 3.56 mm to (228.9, 59.4)
- moved P23 3.56 mm to (228.9, 40.1)
- moved RV2 3.30 mm to (142.7, 71.4)
- moved 3mm_hole 2.54 mm to (238.8, 83.8)
- moved 3mm_hole 2.54 mm to (238.8, 20.3)
- moved D9 2.29 mm to (236.7, 49.5)
- moved R62 2.29 mm to (231.9, 49.5)
- moved R37 1.37 mm to (159.0, 26.7), turned to 270 degrees
- moved R41 1.08 mm to (160.8, 25.1), turned to 90 degrees
Connections:
- D9 pad 1: N-0000065 (its old number) -> N-0000027
- F2 pad 1: N-0000042 (its old number) -> N-0000027
- P19 pad 1: CTRL_GND -> N-0000086
- P23 pad 1: N-0000065 (its old number) -> N-0000027
- R37 pad 2: CTRL_GND -> N-0000086
- R41 pad 1: CTRL_GND -> N-0000086
- R64 pad 1: N-0000042 (its old number) -> N-0000086
- R64 pad 2: N-0000065 (its old number) -> CTRL_GND
- U12 pad 12: N-0000065 (its old number) -> N-0000086
- U12 pad 14: N-0000042 (its old number) -> CTRL_GND
- U13 pad 12: N-0000042 (its old number) -> CTRL_GND
- U13 pad 14: N-0000065 (its old number) -> N-0000086
Routing:
- net N-0000086: track 0.00 -> 226.9 mm, vias 0 -> 6
- net N-0000065 (its old number): track 147.7 -> 0.00 mm, vias 4 -> 0
- net N-0000042 (its old number): track 125.1 -> 0.00 mm, vias 2 -> 0
- net N-0000027: track 0.00 -> 41.3 mm
- net CTRL_GND: track 158.7 -> 192.2 mm, vias 32 -> 33
- net N-0000022: track 77.7 -> 80.7 mm
- net N-0000074: track 4.96 -> 7.67 mm
- net N-0000096: track 25.5 -> 28.0 mm
- net N-0000010: track 181.9 -> 183.4 mm
- net IC_POW-: track 362.8 -> 364.3 mm
- net IC_POW+: track 447.3 -> 448.6 mm
- net N-0000044: track 192.1 -> 193.1 mm
- net N-0000018: track 15.9 -> 16.5 mm
Other:
- board size 236.5 x 74.2 mm -> 232.7 x 74.2 mm
- board text added: "Reg V+"
- board text removed: "GND"
- board text removed: "reg V"
