File: $DCMGv2SOURCEStest.sch (KiCad schematic (older format))
At the start: 165 parts, among them P10 NC_SCGR_SIG, P14 UNREG_V_SIG, P15 UNREG_I_SIG, P16 TO_REG+, P17 TO_REG-, P18 FROM_REG+, P19 FROM_REG-, P20 REG_V_SIG, P21 TO_GRID-, P22 REG_I_SIG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

Commit message: added optional filtering capacitors for measurement amplifiers. corrected zener clamps to clamp high AND low voltages.
Parts:
- added C10, C3, C4, C5, C9: C, ~, symbol C
- added D15, D17, D18, D19: BZX84C10L, ~, symbol ZENER
Connections:
- wire segments 435 -> 455
